File: esp-rgb-controller.kicad_pcb (KiCad board)
At the start: 2 copper layers, 57.2 x 31.8 mm, 31 parts, among them J1 Barrel_Jack_Switch, J2 SPARE_GPIO, J3 MCU_UART, J4 AVR-ISP-6, J5 ESP_UART, J6 STRIP, Q1 DMG4800LK3, Q2 DMG4800LK3, Q3 DMG4800LK3, U1 ATmega328P-AU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

Commit message: more PCB work
Parts:
- F1: moved to B.Cu
- moved F1 35.1 mm to (168.1, 118.1), turned to 0 degrees
Routing:
- net +12V: track 0.00 -> 15.2 mm
- net /G: track 0.00 -> 9.90 mm
- net /R: track 0.00 -> 8.69 mm
- net /B: track 0.00 -> 8.59 mm

Commit message: more schematic + pcb work
Parts:
- removed J2: SPARE_GPIO, Connector_PinHeader_2.54mm:PinHeader_1x05_P2.54mm_Vertical
- removed J3: MCU_UART, Connector_PinHeader_2.54mm:PinHeader_1x04_P2.54mm_Vertical
- removed J5: ESP_UART, Connector_PinHeader_2.54mm:PinHeader_1x04_P2.54mm_Vertical
- removed JP1, JP2: UART_VCC, Connector_PinHeader_2.54mm:PinHeader_1x02_P2.54mm_Vertical
- added REF**: MountingHole_2.1mm, MountingHole:MountingHole_2.1mm, F.Cu at (128.9, 119.4)
- added REF**: MountingHole_2.1mm, MountingHole:MountingHole_2.1mm, F.Cu at (128.9, 92.7)
- added REF**: MountingHole_2.1mm, MountingHole:MountingHole_2.1mm, F.Cu at (187.3, 92.7)
- added REF**: MountingHole_2.1mm, MountingHole:MountingHole_2.1mm, F.Cu at (187.3, 119.4)
- C4, R3, R4, R5: moved to B.Cu
- J4: footprint Connector_PinHeader_2.54mm:PinHeader_2x03_P2.54mm_Vertical -> Connector_PinHeader_2.54mm:PinHeader_2x03_P2.54mm_Vertical_SMD
- moved R3 66.7 mm to (168.9, 110.2), turned to 90 degrees
- moved D1 65.5 mm to (157.7, 93.6), turned to 225 degrees
- moved C1 63.1 mm to (146.1, 118.9)
- moved R2 62.5 mm to (134.9, 118.7), turned to 180 degrees
- moved R4 57.3 mm to (168.9, 102.5), turned to 90 degrees
- moved R5 54.9 mm to (168.9, 94.6), turned to 90 degrees
- moved C4 48.8 mm to (161.2, 99.8), turned to 180 degrees
- moved R1 42.6 mm to (155.7, 92.3), turned to 45 degrees
- moved D2 22.9 mm to (134.3, 115.6), turned to 0 degrees
- moved U3 14.2 mm to (142.2, 115.6), turned to 90 degrees
- moved C6 12.9 mm to (149.9, 100.3)
- moved C3 12.8 mm to (146.2, 91.9)
- moved U2 12.8 mm to (142.9, 95.0)
- moved L1 12.8 mm to (149.7, 95.5)
- moved C2 12.7 mm to (142.2, 100.3)
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Routing:
- net Net-(F1-Pad1): track 0.00 -> 58.1 mm
- net +3V3: track 0.00 -> 22.3 mm, vias 0 -> 1
- net R_PWM: track 0.00 -> 15.9 mm, vias 0 -> 1
- net +12V: track 15.2 -> 0.00 mm
- net G_PWM: track 0.00 -> 13.7 mm, vias 0 -> 1
- net B_PWM: track 0.00 -> 8.17 mm, vias 0 -> 1
- net Net-(R1-Pad1): track 0.00 -> 6.29 mm
- net Net-(C2-Pad1): track 0.00 -> 5.56 mm
- net Net-(D1-Pad1): track 0.00 -> 2.75 mm
- net /B: track 8.59 -> 10.3 mm
- added copper zone on B.Cu, net +12V
- added copper zone on B.Cu, net GND
- added copper zone on F.Cu, net Net-(C3-Pad2)
- removed copper zone on F.Cu, net Net-(F1-Pad1)
Other:
- board size 57.2 x 31.8 mm -> 63.5 x 31.8 mm

Commit message: finished up design, ordered
Parts:
- removed JP3: GPIO0, Connector_PinHeader_2.54mm:PinHeader_1x02_P2.54mm_Vertical
- added R6: 10k, Resistor_SMD:R_0805_2012Metric_Pad1.15x1.40mm_HandSolder, F.Cu at (152.5, 118.9)
- added TP1: MCU_RX, TestPoint:TestPoint_Pad_D1.0mm, F.Cu at (151.1, 107.3)
- added TP2: MCU_TX, TestPoint:TestPoint_Pad_D1.0mm, F.Cu at (151.1, 109.3)
- added TP3: GND, TestPoint:TestPoint_Pad_D1.0mm, F.Cu at (146.1, 109.3)
- added TP4: 3V3, TestPoint:TestPoint_Pad_D1.0mm, F.Cu at (146.1, 107.3)
- C2: footprint Capacitor_SMD:CP_Elec_5x5.3 -> Capacitor_Tantalum_SMD:CP_EIA-3528-15_AVX-H_Pad1.50x2.35mm_HandSolder
- C4, Q1, Q2, Q3, R3, R4, R5: moved to F.Cu
- C5, C6: footprint Capacitor_SMD:CP_Elec_4x4.5 -> Capacitor_Tantalum_SMD:CP_EIA-3528-15_AVX-H_Pad1.50x2.35mm_HandSolder
- D1, D2: footprint LED_SMD:LED_1206_3216Metric_Pad1.42x1.75mm_HandSolder -> LED_SMD:LED_0805_2012Metric_Pad1.15x1.40mm_HandSolder
- L1: footprint Inductor_SMD:L_Taiyo-Yuden_NR-40xx_HandSoldering -> Inductor_SMD:L_Bourns-SRN6028
- moved C4 7.42 mm to (165.3, 106.0), turned to 225 degrees
- moved R2 6.36 mm to (141.2, 118.9)
- moved D1 5.77 mm to (163.4, 92.8), turned to 315 degrees
- moved D2 3.92 mm to (136.4, 118.9)
- moved R1 2.22 mm to (157.9, 92.8)
- moved F1 2.12 mm to (175.9, 116.8)
- moved C2 1.53 mm to (143.3, 99.2)
- moved C5 1.02 mm to (150.0, 104.4)
- moved U1 0.99 mm to (160.7, 100.5)
- moved J4 0.90 mm to (160.7, 113.0), turned to 0 degrees
- moved R3 0.68 mm to (169.5, 110.5), turned to 270 degrees
- moved C6 0.65 mm to (150.0, 101.0)
- moved R4 0.64 mm to (169.5, 102.5), turned to 270 degrees
- moved R5 0.64 mm to (169.5, 94.6), turned to 270 degrees
- moved U2 0.63 mm to (143.3, 94.5)
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Connections:
- U1 pad 10: B_PWM -> R_PWM
- U1 pad 13: R_PWM -> B_PWM
Routing:
- net +3V3: track 22.3 -> 103.3 mm, vias 1 -> 2
- net Net-(F1-Pad1): track 58.1 -> 9.98 mm
- net ~RST: track 0.00 -> 25.0 mm, vias 0 -> 2
- net ESP_TX: track 0.00 -> 23.5 mm, vias 0 -> 1
- net MOSI: track 0.00 -> 19.9 mm, vias 0 -> 2
- net SCK: track 0.00 -> 18.7 mm, vias 0 -> 2
- net MISO: track 0.00 -> 17.2 mm, vias 0 -> 2
- net ESP_RX: track 0.00 -> 15.0 mm
- net Net-(R6-Pad1): track 0.00 -> 9.99 mm, vias 0 -> 1
- net MCU_TX: track 0.00 -> 9.79 mm
- net GND: track 0.00 -> 8.88 mm, vias 0 -> 8
- net MCU_RX: track 0.00 -> 8.61 mm
- net /R: track 9.12 -> 15.3 mm
- net /G: track 9.48 -> 15.7 mm
- net /B: track 10.3 -> 16.4 mm
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- added copper zone on B.Cu, net Net-(F1-Pad1)
Other:
- rule trace_min: 0.2 -> 0.127
- rule via_min_size: 0.4 -> 0.6096
- board text added: "12V"
- board text added: "3V3"
- board text added: "4A"
- board text added: "500mA"
- board text added: "B"
- board text added: "G"
- board text added: "GND"
- board text added: "R"
- board text added: "RX"
- board text added: "TX"
- board text added: "W3AXL Wifi RGB Controller rev A / 10-21-2020"
